Commit message: getting ready to collect all nescessary data

File: robotarm2/urdf/arm.urdf (robot description, URDF)
Before this commit: robot arm, 6 links, 5 joints
Joints:
- joint link_Cube.001: origin xyz=0 0 0.26166 rpy=1.5708 -0.7854 0 -> xyz=0 0 0.26166 rpy=1.5708 0 0
- joint link_Cube.002: axis 0 0 1.0 -> 0 -1.0 0; origin xyz=0 0.84553 0 rpy=0 0 -0.7854 -> xyz=0 0.84553 0 rpy=-1.5708 0 -0.7854
- joint link_Cube.003: axis 0 0 1.0 -> 0 -1.0 0; origin xyz=0 0.844 0 rpy=0 0 -0.71217 -> xyz=-0.5968 0 0.5968 rpy=0 -0.7854 0
- joint link_Cube.004: origin xyz=0 0.91888 0 rpy=-1.5708 0 0 -> xyz=0 0 0.91888 rpy=0 0 0
